File: 555 Breathing LED v2.sch (KiCad schematic (older format))
At the start: 10 parts, among them Q1 PN2222A, U1 LMC555xN

Commit message: update
Parts:
- added BT1: Battery_Cell, Battery:BatteryHolder_Keystone_107_1x23mm, symbol Device:Battery_Cell
Connections:
- net GND: now also BT1.2 (-)
- net VCC: now also BT1.1 (+)
Changed lines of the file:
@@
 	0    -1   -1   0
 $EndComp
+$Comp
+L Device:Battery_Cell BT1
+U 1 1 6141E819
+P 3800 3250
+F 0 "BT1" H 3918 3346 50  0000 L CNN
+F 1 "Battery_Cell" H 3918 3255 50  0000 L CNN
+F 2 "Battery:BatteryHolder_Keystone_107_1x23mm" V 3800 3310 50  0001 C CNN
+F 3 "~" V 3800 3310 50  0001 C CNN
+	1    3800 3250
+	1    0    0    -1
+$EndComp
+$Comp
+L power:VCC #PWR?
+U 1 1 61421A93
+P 3800 2500
+F 0 "#PWR?" H 3800 2350 50  0001 C CNN
+F 1 "VCC" H 3815 2673 50  0000 C CNN
+F 2 "" H 3800 2500 50  0001 C CNN
+F 3 "" H 3800 2500 50  0001 C CNN
+	1    3800 2500
+	1    0    0    -1
+$EndComp
+$Comp
+L power:GND #PWR?
+U 1 1 614228AA
+P 3800 4150
+F 0 "#PWR?" H 3800 3900 50  0001 C CNN
+F 1 "GND" H 3805 3977 50  0000 C CNN
+F 2 "" H 3800 4150 50  0001 C CNN
+F 3 "" H 3800 4150 50  0001 C CNN
+	1    3800 4150
+	1    0    0    -1
+$EndComp
+Wire Wire Line
+	3800 3350 3800 4150
+Wire Wire Line
+	3800 2500 3800 3050
 $EndSCHEMATC

Commit message: Updated Schematic
Parts:
- added R5: 10k, Potentiometer_THT:Potentiometer_Bourns_PTA2043_Single_Slide, symbol Device:R_POT_US
- R4: value 22k -> 10k
Connections:
- net at C2.1, U1.2 (TR), U1.6 (THR): now also R5.2; no longer R4.2
- net out: now reaches R1.1, U1.3 (Q)
- new net: R4.2, R5.1
Other:
- note added: "100 ohm for Green LED"
- note added: "220 ohm for Red, Yellow, White, and Blue LED"
- note added: "R2 Note"
- moved on the sheet: C1, C2, D1, Q1, R1, R2, R3, R4
Changed lines of the file:
@@
 L Transistor_BJT:PN2222A Q1
 U 1 1 613D51FA
-P 7000 3050
-F 0 "Q1" H 7190 3096 50  0000 L CNN
-F 1 "PN2222A" H 7190 3005 50  0000 L CNN
-F 2 "Package_TO_SOT_THT:TO-92L_Wide" H 7200 2975 50  0001 L CIN
-F 3 "https://www.onsemi.com/pub/Collateral/PN2222-D.PDF" H 7000 3050 50  0001 L CNN
-	1    7000 3050
+P 8150 3050
+F 0 "Q1" H 8340 3096 50  0000 L CNN
+F 1 "PN2222A" H 8340 3005 50  0000 L CNN
+F 2 "Package_TO_SOT_THT:TO-92L_Wide" H 8350 2975 50  0001 L CIN
+F 3 "https://www.onsemi.com/pub/Collateral/PN2222-D.PDF" H 8150 3050 50  0001 L CNN
+	1    8150 3050
 	1    0    0    -1
 $EndComp
@@
 L Device:CP1 C1
 U 1 1 613D8B54
-P 6700 3500
-F 0 "C1" H 6815 3546 50  0000 L CNN
-F 1 "47uF" H 6815 3455 50  0000 L CNN
-F 2 "Capacitor_THT:CP_Radial_D6.3mm_P2.50mm" H 6700 3500 50  0001 C CNN
-F 3 "~" H 6700 3500 50  0001 C CNN
-	1    6700 3500
+P 7850 3500
+F 0 "C1" H 7965 3546 50  0000 L CNN
+F 1 "47uF" H 7965 3455 50  0000 L CNN
+F 2 "Capacitor_THT:CP_Radial_D6.3mm_P2.50mm" H 7850 3500 50  0001 C CNN
+F 3 "~" H 7850 3500 50  0001 C CNN
+	1    7850 3500
 	1    0    0    -1
 $EndComp
@@
 L Device:R_US R2
 U 1 1 613E13B4
-P 7100 3800
-F 0 "R2" H 7168 3846 50  0000 L CNN
-F 1 "220" H 7168 3755 50  0000 L CNN
-F 2 "Resistor_THT:R_Axial_DIN0309_L9.0mm_D3.2mm_P12.70mm_Horizontal" V 7140 3790 50  0001 C CNN
-F 3 "~" H 7100 3800 50  0001 C CNN
-	1    7100 3800
+P 8250 3800
+F 0 "R2" H 8318 3799 50  0000 L CNN
+F 1 "220" H 8318 3755 50  0001 L CNN
+F 2 "Resistor_THT:R_Axial_DIN0309_L9.0mm_D3.2mm_P12.70mm_Horizontal" V 8290 3790 50  0001 C CNN
+F 3 "~" H 8250 3800 50  0001 C CNN
+	1    8250 3800
 	1    0    0    -1
 $EndComp
@@
 L power:GND #PWR?
 U 1 1 613E23F8
-P 7100 4150
-F 0 "#PWR?" H 7100 3900 50  0001 C CNN
-F 1 "GND" H 7105 3977 50  0000 C CNN
-F 2 "" H 7100 4150 50  0001 C CNN
-F 3 "" H 7100 4150 50  0001 C CNN
-	1    7100 4150
+P 8250 4150
+F 0 "#PWR?" H 8250 3900 50  0001 C CNN
+F 1 "GND" H 8255 3977 50  0000 C CNN
+F 2 "" H 8250 4150 50  0001 C CNN
+F 3 "" H 8250 4150 50  0001 C CNN
+	1    8250 4150
 	1    0    0    -1
 $EndComp
@@
 L power:GND #PWR?
 U 1 1 613E5215
-P 6700 4150
-F 0 "#PWR?" H 6700 3900 50  0001 C CNN
-F 1 "GND" H 6705 3977 50  0000 C CNN
-F 2 "" H 6700 4150 50  0001 C CNN
-F 3 "" H 6700 4150 50  0001 C CNN
-	1    6700 4150
+P 7850 4150
+F 0 "#PWR?" H 7850 3900 50  0001 C CNN
+F 1 "GND" H 7855 3977 50  0000 C CNN
+F 2 "" H 7850 4150 50  0001 C CNN
+F 3 "" H 7850 4150 50  0001 C CNN
+	1    7850 4150
 	1    0    0    -1
 $EndComp
@@
 L Device:LED D1
 U 1 1 613E992B
-P 7100 3450
-F 0 "D1" V 7139 3332 50  0000 R CNN
-F 1 "LED" V 7048 3332 50  0000 R CNN
-F 2 "LED_THT:LED_D10.0mm" H 7100 3450 50  0001 C CNN
-F 3 "~" H 7100 3450 50  0001 C CNN
-	1    7100 3450
+P 8250 3450
+F 0 "D1" V 8289 3332 50  0000 R CNN
+F 1 "LED" V 8198 3332 50  0000 R CNN
+F 2 "LED_THT:LED_D10.0mm" H 8250 3450 50  0001 C CNN
+F 3 "~" H 8250 3450 50  0001 C CNN
+	1    8250 3450
 	0    -1   -1   0
 $EndComp
 Wire Wire Line
-	7100 3250 7100 3300
-Wire Wire Line
-	7100 3600 7100 3650
-Wire Wire Line
-	6600 3050 6700 3050
-Connection ~ 6700 3050
-Wire Wire Line
-	6700 3050 6800 3050
-Wire Wire Line
-	6700 3050 6700 3350
+	8250 3250 8250 3300
+Wire Wire Line
+	8250 3600 8250 3650
+Wire Wire Line
+	7750 3050 7850 3050
+Connection ~ 7850 3050
+Wire Wire Line
+	7850 3050 7950 3050
+Wire Wire Line
+	7850 3050 7850 3350
 $Comp
 L Device:R_US R3
 U 1 1 613F32B6
-P 5900 2750
-F 0 "R3" H 5968 2796 50  0000 L CNN
-F 1 "2k2" H 5968 2705 50  0000 L CNN
-F 2 "Resistor_THT:R_Axial_DIN0309_L9.0mm_D3.2mm_P12.70mm_Horizontal" V 5940 2740 50  0001 C CNN
-F 3 "~" H 5900 2750 50  0001 C CNN
-	1    5900 2750
+P 6000 2750
+F 0 "R3" H 6068 2796 50  0000 L CNN
+F 1 "2k2" H 6068 2705 50  0000 L CNN
+F 2 "Resistor_THT:R_Axial_DIN0309_L9.0mm_D3.2mm_P12.70mm_Horizontal" V 6040 2740 50  0001 C CNN
+F 3 "~" H 6000 2750 50  0001 C CNN
+	1    6000 2750
 	1    0    0    -1
 $EndComp
@@
 L Device:R_US R4
 U 1 1 613F3F7C
-P 5900 3450
-F 0 "R4" H 5968 3496 50  0000 L CNN
-F 1 "22k" H 5968 3405 50  0000 L CNN
-F 2 "Resistor_THT:R_Axial_DIN0309_L9.0mm_D3.2mm_P12.70mm_Horizontal" V 5940 3440 50  0001 C CNN
-F 3 "~" H 5900 3450 50  0001 C CNN
-	1    5900 3450
-	1    0    0    -1
-$EndComp
-Wire Wire Line
-	5700 3050 6300 3050
+P 6250 3250
+F 0 "R4" H 6318 3296 50  0000 L CNN
+F 1 "10k" H 6318 3205 50  0000 L CNN
+F 2 "Resistor_THT:R_Axial_DIN0309_L9.0mm_D3.2mm_P12.70mm_Horizontal" V 6290 3240 50  0001 C CNN
+F 3 "~" H 6250 3250 50  0001 C CNN
+	1    6250 3250
+	0    -1   -1   0
+$EndComp
 $Comp
 L power:VCC #PWR?
 U 1 1 613FD065
-P 5900 2500
-F 0 "#PWR?" H 5900 2350 50  0001 C CNN
-F 1 "VCC" H 5915 2673 50  0000 C CNN
-F 2 "" H 5900 2500 50  0001 C CNN
-F 3 "" H 5900 2500 50  0001 C CNN
-	1    5900 2500
+P 6000 2500
+F 0 "#PWR?" H 6000 2350 50  0001 C CNN
+F 1 "VCC" H 6015 2673 50  0000 C CNN
+F 2 "" H 6000 2500 50  0001 C CNN
+F 3 "" H 6000 2500 50  0001 C CNN
+	1    6000 2500
 	1    0    0    -1
 $EndComp
@@
 L power:VCC #PWR?
 U 1 1 613FDD9B
-P 7100 2500
-F 0 "#PWR?" H 7100 2350 50  0001 C CNN
-F 1 "VCC" H 7115 2673 50  0000 C CNN
-F 2 "" H 7100 2500 50  0001 C CNN
-F 3 "" H 7100 2500 50  0001 C CNN
-	1    7100 2500
-	1    0    0    -1
-$EndComp
-Wire Wire Line
-	5900 2500 5900 2600
+P 8250 2500
+F 0 "#PWR?" H 8250 2350 50  0001 C CNN
+F 1 "VCC" H 8265 2673 50  0000 C CNN
+F 2 "" H 8250 2500 50  0001 C CNN
+F 3 "" H 8250 2500 50  0001 C CNN
+	1    8250 2500
+	1    0    0    -1
+$EndComp
+Wire Wire Line
+	6000 2500 6000 2600
 Wire Wire Line
 	4550 2500 4550 2750
 Wire Wire Line
-	7100 2500 7100 2850
+	8250 2500 8250 2850
 $Comp
 L Device:CP1 C2
 U 1 1 613FFFB8
-P 5900 3950
-F 0 "C2" H 6015 3996 50  0000 L CNN
-F 1 "47uF" H 6015 3905 50  0000 L CNN
-F 2 "Capacitor_THT:CP_Radial_D6.3mm_P2.50mm" H 5900 3950 50  0001 C CNN
-F 3 "~" H 5900 3950 50  0001 C CNN
-	1    5900 3950
+P 6050 3950
+F 0 "C2" H 6165 3996 50  0000 L CNN
+F 1 "47uF" H 6165 3905 50  0000 L CNN
+F 2 "Capacitor_THT:CP_Radial_D6.3mm_P2.50mm" H 6050 3950 50  0001 C CNN
+F 3 "~" H 6050 3950 50  0001 C CNN
+	1    6050 3950
 	1    0    0    -1
 $EndComp
@@
 L power:GND #PWR?
 U 1 1 61400FBF
-P 5900 4150
-F 0 "#PWR?" H 5900 3900 50  0001 C CNN
-F 1 "GND" H 5905 3977 50  0000 C CNN
-F 2 "" H 5900 4150 50  0001 C CNN
-F 3 "" H 5900 4150 50  0001 C CNN
-	1    5900 4150
-	1    0    0    -1
-$EndComp
-Wire Wire Line
-	5900 3600 5900 3700
+P 6050 4150
+F 0 "#PWR?" H 6050 3900 50  0001 C CNN
+F 1 "GND" H 6055 3977 50  0000 C CNN
+F 2 "" H 6050 4150 50  0001 C CNN
+F 3 "" H 6050 4150 50  0001 C CNN
+	1    6050 4150
+	1    0    0    -1
+$EndComp
 Wire Wire Line
 	4600 3250 4600 3800
 Wire Wire Line
 	4600 4100 4600 4150
-Wire Wire Line
-	5700 3700 5900 3700
 Wire Wire Line
 	5700 3450 5700 3700
@@
 Connection ~ 5700 3700
 Wire Wire Line
-	5900 3700 5900 3800
-Connection ~ 5900 3700
-Wire Wire Line
 	5200 3650 5200 4150
 Wire Wire Line
-	5900 4150 5900 4100
-Wire Wire Line
-	6700 3650 6700 4150
-Wire Wire Line
-	7100 3950 7100 4150
-Wire Wire Line
-	5900 2900 5900 3250
-Wire Wire Line
-	5700 3250 5900 3250
-Connection ~ 5900 3250
-Wire Wire Line
-	5900 3250 5900 3300
+	6050 4150 6050 4100
+Wire Wire Line
+	7850 3650 7850 4150
+Wire Wire Line
+	8250 3950 8250 4150
+Wire Wire Line
+	6000 2900 6000 3250
 $Comp
 L Device:R_US R1
 U 1 1 613D6DC9
-P 6450 3050
-F 0 "R1" V 6614 3012 50  0000 L CNN
-F 1 "2k2" V 6535 2992 50  0000 L CNN
-F 2 "Resistor_THT:R_Axial_DIN0309_L9.0mm_D3.2mm_P12.70mm_Horizontal" V 6490 3040 50  0001 C CNN
-F 3 "~" H 6450 3050 50  0001 C CNN
-	1    6450 3050
+P 7600 3050
+F 0 "R1" V 7764 3012 50  0000 L CNN
+F 1 "2k2" V 7685 2992 50  0000 L CNN
+F 2 "Resistor_THT:R_Axial_DIN0309_L9.0mm_D3.2mm_P12.70mm_Horizontal" V 7640 3040 50  0001 C CNN
+F 3 "~" H 7600 3050 50  0001 C CNN
+	1    7600 3050
 	0    -1   -1   0
 $EndComp
@@
 Wire Wire Line
 	3800 2500 3800 3050
+Text Notes 7200 4700 0    50   ~ 0
+220 ohm for Red, Yellow, White, and Blue LED
+Text Notes 7200 4800 0    50   ~ 0
+100 ohm for Green LED
+Text Notes 7200 4600 0    50   ~ 0
+R2 Note
+$Comp
+L Device:R_POT_US R5
+U 1 1 6141A453
+P 6550 3700
+F 0 "R5" H 6482 3746 50  0000 R CNN
+F 1 "10k" H 6482 3655 50  0000 R CNN
+F 2 "Potentiometer_THT:Potentiometer_Bourns_PTA2043_Single_Slide" H 6550 3700 50  0001 C CNN
+F 3 "~" H 6550 3700 50  0001 C CNN
+	1    6550 3700
+	-1   0    0    -1
+$EndComp
+Text GLabel 7300 3050 0    50   Input ~ 0
+out
+Text GLabel 5700 3050 2    50   Input ~ 0
+out
+Wire Wire Line
+	5700 3250 6000 3250
+Wire Wire Line
+	7300 3050 7450 3050
+Wire Wire Line
+	6050 3700 6050 3800
+Wire Wire Line
+	5700 3700 6050 3700
+Wire Wire Line
+	6100 3250 6000 3250
+Connection ~ 6000 3250
+Wire Wire Line
+	6400 3250 6550 3250
+Wire Wire Line
+	6550 3250 6550 3550
+Wire Wire Line
+	6400 3700 6050 3700
+Connection ~ 6050 3700
 $EndSCHEMATC

Commit message: updated schematic
Parts:
- C1: value 47uF -> 220uF
Changed lines of the file:
@@
 P 7850 3500
 F 0 "C1" H 7965 3546 50  0000 L CNN
-F 1 "47uF" H 7965 3455 50  0000 L CNN
+F 1 "220uF" H 7965 3455 50  0000 L CNN
 F 2 "Capacitor_THT:CP_Radial_D6.3mm_P2.50mm" H 7850 3500 50  0001 C CNN
 F 3 "~" H 7850 3500 50  0001 C CNN

Commit message: updated footprint of C3
Parts:
- C3: footprint (none) -> Capacitor_THT:C_Disc_D5.0mm_W2.5mm_P2.50mm
Changed lines of the file:
@@
 F 0 "C3" H 4715 3996 50  0000 L CNN
 F 1 "0.1uF" H 4715 3905 50  0000 L CNN
-F 2 "" H 4638 3800 50  0001 C CNN
+F 2 "Capacitor_THT:C_Disc_D5.0mm_W2.5mm_P2.50mm" H 4638 3800 50  0001 C CNN
 F 3 "~" H 4600 3950 50  0001 C CNN
 	1    4600 3950

Commit message: Finished PCB
Parts:
- added SW1: SW_SPDT, 555-Breathing-LED-v2:MHS12204_SPDT, symbol Switch:SW_SPDT
- BT1: footprint Battery:BatteryHolder_Keystone_107_1x23mm -> 555-Breathing-LED-v2:BatteryHolder_MPD_BA9VPC_1xPP3noholes
Connections:
- net VCC: now also SW1.2 (B); no longer BT1.1 (+)
- new net: BT1.1 (+), SW1.1 (A)
Other:
- moved on the sheet: BT1
Changed lines of the file:
@@
 $EndComp
 $Comp
-L power:GND #PWR?
+L power:GND #PWR0101
 U 1 1 613D32FA
 P 4600 4150
-F 0 "#PWR?" H 4600 3900 50  0001 C CNN
+F 0 "#PWR0101" H 4600 3900 50  0001 C CNN
 F 1 "GND" H 4605 3977 50  0000 C CNN
 F 2 "" H 4600 4150 50  0001 C CNN
@@
 $EndComp
 $Comp
-L power:VCC #PWR?
+L power:VCC #PWR0102
 U 1 1 613D3531
 P 4550 2500
-F 0 "#PWR?" H 4550 2350 50  0001 C CNN
+F 0 "#PWR0102" H 4550 2350 50  0001 C CNN
 F 1 "VCC" H 4565 2673 50  0000 C CNN
 F 2 "" H 4550 2500 50  0001 C CNN
@@
 	4700 3250 4600 3250
 $Comp
-L power:GND #PWR?
+L power:GND #PWR0103
 U 1 1 613DFB38
 P 5200 4150
-F 0 "#PWR?" H 5200 3900 50  0001 C CNN
+F 0 "#PWR0103" H 5200 3900 50  0001 C CNN
 F 1 "GND" H 5205 3977 50  0000 C CNN
 F 2 "" H 5200 4150 50  0001 C CNN
@@
 $EndComp
 $Comp
-L power:GND #PWR?
+L power:GND #PWR0104
 U 1 1 613E23F8
 P 8250 4150
-F 0 "#PWR?" H 8250 3900 50  0001 C CNN
+F 0 "#PWR0104" H 8250 3900 50  0001 C CNN
 F 1 "GND" H 8255 3977 50  0000 C CNN
 F 2 "" H 8250 4150 50  0001 C CNN
@@
 $EndComp
 $Comp
-L power:GND #PWR?
+L power:GND #PWR0105
 U 1 1 613E5215
 P 7850 4150
-F 0 "#PWR?" H 7850 3900 50  0001 C CNN
+F 0 "#PWR0105" H 7850 3900 50  0001 C CNN
 F 1 "GND" H 7855 3977 50  0000 C CNN
 F 2 "" H 7850 4150 50  0001 C CNN
@@
 $EndComp
 $Comp
-L power:VCC #PWR?
+L power:VCC #PWR0106
 U 1 1 613FD065
 P 6000 2500
-F 0 "#PWR?" H 6000 2350 50  0001 C CNN
+F 0 "#PWR0106" H 6000 2350 50  0001 C CNN
 F 1 "VCC" H 6015 2673 50  0000 C CNN
 F 2 "" H 6000 2500 50  0001 C CNN
@@
 $EndComp
 $Comp
-L power:VCC #PWR?
+L power:VCC #PWR0107
 U 1 1 613FDD9B
 P 8250 2500
-F 0 "#PWR?" H 8250 2350 50  0001 C CNN
+F 0 "#PWR0107" H 8250 2350 50  0001 C CNN
 F 1 "VCC" H 8265 2673 50  0000 C CNN
 F 2 "" H 8250 2500 50  0001 C CNN
@@
 $EndComp
 $Comp
-L power:GND #PWR?
+L power:GND #PWR0108
 U 1 1 61400FBF
 P 6050 4150
-F 0 "#PWR?" H 6050 3900 50  0001 C CNN
+F 0 "#PWR0108" H 6050 3900 50  0001 C CNN
 F 1 "GND" H 6055 3977 50  0000 C CNN
 F 2 "" H 6050 4150 50  0001 C CNN
@@
 L Device:Battery_Cell BT1
 U 1 1 6141E819
-P 3800 3250
-F 0 "BT1" H 3918 3346 50  0000 L CNN
-F 1 "Battery_Cell" H 3918 3255 50  0000 L CNN
-F 2 "Battery:BatteryHolder_Keystone_107_1x23mm" V 3800 3310 50  0001 C CNN
-F 3 "~" V 3800 3310 50  0001 C CNN
-	1    3800 3250
-	1    0    0    -1
-$EndComp
-$Comp
-L power:VCC #PWR?
+P 3800 3600
+F 0 "BT1" H 3918 3696 50  0000 L CNN
+F 1 "Battery_Cell" H 3918 3605 50  0000 L CNN
+F 2 "555-Breathing-LED-v2:BatteryHolder_MPD_BA9VPC_1xPP3noholes" V 3800 3660 50  0001 C CNN
+F 3 "~" V 3800 3660 50  0001 C CNN
+	1    3800 3600
+	1    0    0    -1
+$EndComp
+$Comp
+L power:VCC #PWR0109
 U 1 1 61421A93
-P 3800 2500
-F 0 "#PWR?" H 3800 2350 50  0001 C CNN
-F 1 "VCC" H 3815 2673 50  0000 C CNN
-F 2 "" H 3800 2500 50  0001 C CNN
-F 3 "" H 3800 2500 50  0001 C CNN
-	1    3800 2500
-	1    0    0    -1
-$EndComp
-$Comp
-L power:GND #PWR?
+P 3700 2500
+F 0 "#PWR0109" H 3700 2350 50  0001 C CNN
+F 1 "VCC" H 3715 2673 50  0000 C CNN
+F 2 "" H 3700 2500 50  0001 C CNN
+F 3 "" H 3700 2500 50  0001 C CNN
+	1    3700 2500
+	1    0    0    -1
+$EndComp
+$Comp
+L power:GND #PWR0110
 U 1 1 614228AA
 P 3800 4150
-F 0 "#PWR?" H 3800 3900 50  0001 C CNN
+F 0 "#PWR0110" H 3800 3900 50  0001 C CNN
 F 1 "GND" H 3805 3977 50  0000 C CNN
 F 2 "" H 3800 4150 50  0001 C CNN
@@
 	1    0    0    -1
 $EndComp
-Wire Wire Line
-	3800 3350 3800 4150
-Wire Wire Line
-	3800 2500 3800 3050
 Text Notes 7200 4700 0    50   ~ 0
 220 ohm for Red, Yellow, White, and Blue LED
@@
 	6400 3700 6050 3700
 Connection ~ 6050 3700
+$Comp
+L Switch:SW_SPDT SW1
+U 1 1 614A4049
+P 3700 2950
+F 0 "SW1" V 3654 3098 50  0000 L CNN
+F 1 "SW_SPDT" V 3745 3098 50  0000 L CNN
+F 2 "555-Breathing-LED-v2:MHS12204_SPDT" H 3700 2950 50  0001 C CNN
+F 3 "~" H 3700 2950 50  0001 C CNN
+	1    3700 2950
+	0    1    1    0
+$EndComp
+Wire Wire Line
+	3700 2500 3700 2750
+Wire Wire Line
+	3800 3150 3800 3400
+Wire Wire Line
+	3800 3700 3800 4150
 $EndSCHEMATC

Commit message: Updated schematic
Parts:
- R2: value 220 -> 100
Other:
- note removed: "100 ohm for Green LED"
- note removed: "220 ohm for Red, Yellow, White, and Blue LED"
- note removed: "R2 Note"
Changed lines of the file:
@@
 P 8250 3800
 F 0 "R2" H 8318 3799 50  0000 L CNN
-F 1 "220" H 8318 3755 50  0001 L CNN
+F 1 "100" H 8318 3720 50  0000 L CNN
 F 2 "Resistor_THT:R_Axial_DIN0309_L9.0mm_D3.2mm_P12.70mm_Horizontal" V 8290 3790 50  0001 C CNN
 F 3 "~" H 8250 3800 50  0001 C CNN
@@
 	1    0    0    -1
 $EndComp
-Text Notes 7200 4700 0    50   ~ 0
-220 ohm for Red, Yellow, White, and Blue LED
-Text Notes 7200 4800 0    50   ~ 0
-100 ohm for Green LED
-Text Notes 7200 4600 0    50   ~ 0
-R2 Note
 $Comp
 L Device:R_POT_US R5
