File: 555 Breathing LED v2.sch (KiCad schematic (older format))
At the start: 13 parts, among them Q1 PN2222A, SW1 SW_SPDT, U1 LMC555xN

Commit message: Updated, epic fortnite
Parts:
- added D2: 1N4148, Diode_THT:D_DO-35_SOD27_P7.62mm_Horizontal, symbol Simulation_SPICE:DIODE
- BT1: footprint 555-Breathing-LED-v2:BatteryHolder_MPD_BA9VPC_1xPP3noholes -> Local:BatteryHolder_MPD_BA9VPC_1xPP3noholes
Connections:
- net at BT1.1 (+): now also D2.1 (A); no longer SW1.1 (A)
- new net: D2.2 (K), SW1.1 (A)
Other:
- moved on the sheet: BT1
Changed lines of the file:
@@
 L Device:Battery_Cell BT1
 U 1 1 6141E819
-P 3150 4250
-F 0 "BT1" H 3268 4346 50  0000 L CNN
-F 1 "Battery_Cell" H 3268 4255 50  0000 L CNN
-F 2 "555-Breathing-LED-v2:BatteryHolder_MPD_BA9VPC_1xPP3noholes" V 3150 4310 50  0001 C CNN
-F 3 "~" V 3150 4310 50  0001 C CNN
-	1    3150 4250
+P 3150 4500
+F 0 "BT1" H 3268 4596 50  0000 L CNN
+F 1 "Battery_Cell" H 3268 4505 50  0000 L CNN
+F 2 "Local:BatteryHolder_MPD_BA9VPC_1xPP3noholes" V 3150 4560 50  0001 C CNN
+F 3 "~" V 3150 4560 50  0001 C CNN
+	1    3150 4500
 	1    0    0    -1
 $EndComp
@@
 F 3 "" H 3050 3150 50  0001 C CNN
 	1    3050 3150
-	1    0    0    -1
-$EndComp
-$Comp
-L power:GND #PWR0110
-U 1 1 614228AA
-P 3150 4800
-F 0 "#PWR0110" H 3150 4550 50  0001 C CNN
-F 1 "GND" H 3155 4627 50  0000 C CNN
-F 2 "" H 3150 4800 50  0001 C CNN
-F 3 "" H 3150 4800 50  0001 C CNN
-	1    3150 4800
 	1    0    0    -1
 $EndComp
@@
 Wire Wire Line
 	3050 3150 3050 3400
+$Comp
+L Simulation_SPICE:DIODE D2
+U 1 1 617C88F4
+P 3150 4050
+F 0 "D2" V 3196 3970 50  0000 R CNN
+F 1 "1N4148" V 3105 3970 50  0000 R CNN
+F 2 "Diode_THT:D_DO-35_SOD27_P7.62mm_Horizontal" H 3150 4050 50  0001 C CNN
+F 3 "~" H 3150 4050 50  0001 C CNN
+F 4 "Y" H 3150 4050 50  0001 L CNN "Spice_Netlist_Enabled"
+F 5 "D" H 3150 4050 50  0001 L CNN "Spice_Primitive"
+	1    3150 4050
+	0    -1   -1   0
+$EndComp
+$Comp
+L power:GND #PWR0110
+U 1 1 614228AA
+P 3150 4800
+F 0 "#PWR0110" H 3150 4550 50  0001 C CNN
+F 1 "GND" H 3155 4627 50  0000 C CNN
+F 2 "" H 3150 4800 50  0001 C CNN
+F 3 "" H 3150 4800 50  0001 C CNN
+	1    3150 4800
+	1    0    0    -1
+$EndComp
 Wire Wire Line
-	3150 3800 3150 4050
+	3150 3900 3150 3800
 Wire Wire Line
-	3150 4350 3150 4800
+	3150 4300 3150 4200
+Wire Wire Line
+	3150 4600 3150 4800
 $EndSCHEMATC

Commit message: fixed diode
Parts:
- D2: symbol Simulation_SPICE:DIODE -> Device:D
Connections:
- net at BT1.1 (+): now also D2.2 (A); no longer D2.1 (A)
- net at SW1.1 (A): now also D2.1 (K); no longer D2.2 (K)
Changed lines of the file:
@@
 	3050 3150 3050 3400
 $Comp
-L Simulation_SPICE:DIODE D2
+L Device:D D2
 U 1 1 617C88F4
 P 3150 4050
@@
 F 5 "D" H 3150 4050 50  0001 L CNN "Spice_Primitive"
 	1    3150 4050
-	0    -1   -1   0
+	0    1    1    0
 $EndComp
 $Comp
